File: joysticks.kicad_sch (KiCad schematic)
At the start: 27 parts, among them J1 DB9_Male_MountingHoles, J2 DB9_Male_MountingHoles, J25 Joystick Ports Mezannine Lower, J26 Joystick Ports Mezannine Upper, SW1 Reset Button, U10 74LS06N, U11 74LS06N, U5 74LS06N, U6 74LVC374, U7 74LVC374, U8 74LS374, U9 74LS374

Commit message: fix many DRC warnings
Parts:
- R17, R18, R19, R20, R21, R22, R23, R24, R25, R26: footprint Resistor_THT:R_Box_L8.4mm_W2.5mm_P5.08mm -> snapeda:Labeled Resistor
Changed lines of the file:
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@@
     (property "Reference" "R22" (id 0) (at 36.83 167.005 90))
     (property "Value" "4K7" (id 1) (at 31.75 168.275 90))
-    (property "Footprint" "Resistor_THT:R_Box_L8.4mm_W2.5mm_P5.08mm" (id 2) (at 31.75 168.275 0)
+    (property "Footprint" "snapeda:Labeled Resistor" (id 2) (at 31.75 168.275 0)
       (effects (font (size 1.27 1.27)) hide)
     )
@@
   (symbol (lib_id "power:GND") (at 104.14 124.46 0) (unit 1)
     (in_bom yes) (on_board yes) (fields_autoplaced)
-    (property "Reference" "#PWR?" (id 0) (at 104.14 130.81 0)
+    (property "Reference" "#PWR0136" (id 0) (at 104.14 130.81 0)
       (effects (font (size 1.27 1.27)) hide)
     )
@@
     (property "Reference" "R20" (id 0) (at 125.095 103.505 90))
     (property "Value" "4K7" (id 1) (at 120.015 104.775 90))
-    (property "Footprint" "Resistor_THT:R_Box_L8.4mm_W2.5mm_P5.08mm" (id 2) (at 120.015 104.775 0)
+    (property "Footprint" "snapeda:Labeled Resistor" (id 2) (at 120.015 104.775 0)
       (effects (font (size 1.27 1.27)) hide)
     )
@@
   (symbol (lib_id "power:GND") (at 104.775 94.615 0) (unit 1)
     (in_bom yes) (on_board yes) (fields_autoplaced)
-    (property "Reference" "#PWR?" (id 0) (at 104.775 100.965 0)
+    (property "Reference" "#PWR0134" (id 0) (at 104.775 100.965 0)
       (effects (font (size 1.27 1.27)) hide)
     )
@@
   (symbol (lib_id "power:GND") (at 104.14 134.62 0) (unit 1)
     (in_bom yes) (on_board yes) (fields_autoplaced)
-    (property "Reference" "#PWR?" (id 0) (at 104.14 140.97 0)
+    (property "Reference" "#PWR0127" (id 0) (at 104.14 140.97 0)
       (effects (font (size 1.27 1.27)) hide)
     )
@@
   (symbol (lib_id "power:GND") (at 34.925 23.495 0) (unit 1)
     (in_bom yes) (on_board yes) (fields_autoplaced)
-    (property "Reference" "#PWR?" (id 0) (at 34.925 29.845 0)
+    (property "Reference" "#PWR0132" (id 0) (at 34.925 29.845 0)
       (effects (font (size 1.27 1.27)) hide)
     )
@@
     (property "Reference" "R17" (id 0) (at 125.095 90.805 90))
     (property "Value" "4K7" (id 1) (at 120.015 92.075 90))
-    (property "Footprint" "Resistor_THT:R_Box_L8.4mm_W2.5mm_P5.08mm" (id 2) (at 120.015 92.075 0)
+    (property "Footprint" "snapeda:Labeled Resistor" (id 2) (at 120.015 92.075 0)
       (effects (font (size 1.27 1.27)) hide)
     )
@@
     (property "Reference" "R19" (id 0) (at 125.095 100.965 90))
     (property "Value" "4K7" (id 1) (at 120.015 102.235 90))
-    (property "Footprint" "Resistor_THT:R_Box_L8.4mm_W2.5mm_P5.08mm" (id 2) (at 120.015 102.235 0)
+    (property "Footprint" "snapeda:Labeled Resistor" (id 2) (at 120.015 102.235 0)
       (effects (font (size 1.27 1.27)) hide)
     )
@@
     (property "Reference" "R26" (id 0) (at 36.83 182.245 90))
     (property "Value" "4K7" (id 1) (at 31.75 183.515 90))
-    (property "Footprint" "Resistor_THT:R_Box_L8.4mm_W2.5mm_P5.08mm" (id 2) (at 31.75 183.515 0)
+    (property "Footprint" "snapeda:Labeled Resistor" (id 2) (at 31.75 183.515 0)
       (effects (font (size 1.27 1.27)) hide)
     )
@@
   (symbol (lib_id "power:GND") (at 53.34 150.495 0) (unit 1)
     (in_bom yes) (on_board yes) (fields_autoplaced)
-    (property "Reference" "#PWR?" (id 0) (at 53.34 156.845 0)
+    (property "Reference" "#PWR0124" (id 0) (at 53.34 156.845 0)
       (effects (font (size 1.27 1.27)) hide)
     )
@@
     (property "Reference" "R21" (id 0) (at 125.095 106.045 90))
     (property "Value" "4K7" (id 1) (at 120.015 107.315 90))
-    (property "Footprint" "Resistor_THT:R_Box_L8.4mm_W2.5mm_P5.08mm" (id 2) (at 120.015 107.315 0)
+    (property "Footprint" "snapeda:Labeled Resistor" (id 2) (at 120.015 107.315 0)
       (effects (font (size 1.27 1.27)) hide)
     )
@@
   (symbol (lib_id "power:GND") (at 78.74 23.495 0) (unit 1)
     (in_bom yes) (on_board yes) (fields_autoplaced)
-    (property "Reference" "#PWR?" (id 0) (at 78.74 29.845 0)
+    (property "Reference" "#PWR0138" (id 0) (at 78.74 29.845 0)
       (effects (font (size 1.27 1.27)) hide)
     )
@@
   (symbol (lib_id "power:GND") (at 141.605 74.295 0) (unit 1)
     (in_bom yes) (on_board yes) (fields_autoplaced)
-    (property "Reference" "#PWR?" (id 0) (at 141.605 80.645 0)
+    (property "Reference" "#PWR0289" (id 0) (at 141.605 80.645 0)
       (effects (font (size 1.27 1.27)) hide)
     )
@@
     (property "Reference" "R24" (id 0) (at 36.83 177.165 90))
     (property "Value" "4K7" (id 1) (at 31.75 178.435 90))
-    (property "Footprint" "Resistor_THT:R_Box_L8.4mm_W2.5mm_P5.08mm" (id 2) (at 31.75 178.435 0)
+    (property "Footprint" "snapeda:Labeled Resistor" (id 2) (at 31.75 178.435 0)
       (effects (font (size 1.27 1.27)) hide)
     )
@@
     (property "Reference" "R18" (id 0) (at 125.095 95.885 90))
     (property "Value" "4K7" (id 1) (at 120.015 97.155 90))
-    (property "Footprint" "Resistor_THT:R_Box_L8.4mm_W2.5mm_P5.08mm" (id 2) (at 120.015 97.155 0)
+    (property "Footprint" "snapeda:Labeled Resistor" (id 2) (at 120.015 97.155 0)
       (effects (font (size 1.27 1.27)) hide)
     )
@@
   (symbol (lib_id "power:GND") (at 58.42 188.595 0) (unit 1)
     (in_bom yes) (on_board yes) (fields_autoplaced)
-    (property "Reference" "#PWR?" (id 0) (at 58.42 194.945 0)
+    (property "Reference" "#PWR0122" (id 0) (at 58.42 194.945 0)
       (effects (font (size 1.27 1.27)) hide)
     )
@@
     (property "Reference" "R23" (id 0) (at 36.83 172.085 90))
     (property "Value" "4K7" (id 1) (at 31.75 173.355 90))
-    (property "Footprint" "Resistor_THT:R_Box_L8.4mm_W2.5mm_P5.08mm" (id 2) (at 31.75 173.355 0)
+    (property "Footprint" "snapeda:Labeled Resistor" (id 2) (at 31.75 173.355 0)
       (effects (font (size 1.27 1.27)) hide)
     )
@@
     (property "Reference" "R25" (id 0) (at 36.83 179.705 90))
     (property "Value" "4K7" (id 1) (at 31.75 180.975 90))
-    (property "Footprint" "Resistor_THT:R_Box_L8.4mm_W2.5mm_P5.08mm" (id 2) (at 31.75 180.975 0)
+    (property "Footprint" "snapeda:Labeled Resistor" (id 2) (at 31.75 180.975 0)
       (effects (font (size 1.27 1.27)) hide)
     )
@@
   (symbol (lib_id "power:GND") (at 16.51 170.815 0) (unit 1)
     (in_bom yes) (on_board yes) (fields_autoplaced)
-    (property "Reference" "#PWR?" (id 0) (at 16.51 177.165 0)
+    (property "Reference" "#PWR0131" (id 0) (at 16.51 177.165 0)
       (effects (font (size 1.27 1.27)) hide)
     )
@@
   (symbol (lib_id "power:GND") (at 146.685 112.395 0) (unit 1)
     (in_bom yes) (on_board yes) (fields_autoplaced)
-    (property "Reference" "#PWR?" (id 0) (at 146.685 118.745 0)
-      (effects (font (size 1.27 1.27)) hide)
-    )
+    (property "Reference" "#PWR0142" (id 0) (at 146.685 118.745 0)
+      (effects (font (size 1.27 1.27)) hide)
+    )
