File: expansionport.kicad_sch (KiCad schematic)
At the start: 18 parts, among them J20 C64_Expansion_Port, U22 74LS06N, U32 74LVC374, U33 74LVC374, U34 74LVC374, U35 74LS374, U36 74LS374, U37 74LS374, U38 74LVC374, U39 74LVC374, U40 74LS374, U41 74LS374, U42 74LS06N

Commit message: address #21 and #22
Parts:
- removed RN3, RN5, RN6: 3.3K x 8, Resistor_THT:R_Array_SIP9, symbol Device:R_Network08
Connections:
- net A0: now also U36.16 (O6); no longer U37.19 (O7)
- net A2: now also U36.2 (O0); no longer U37.5 (O1)
- net A3: now also U36.12 (O4); no longer U36.16 (O6)
- net A6: now also U36.15 (O5); no longer U37.9 (O3)
- net D0: now also U37.5 (O1); no longer U36.2 (O0)
- net D3: now also U37.19 (O7); no longer U36.15 (O5)
- net D7: now also U37.9 (O3); no longer U36.12 (O4)
- net GND: no longer U36.1 (OE), U37.1 (OE), U41.1 (OE)
- net R_W: now also U37.1 (OE)
- net ADDR_EN: now reaches U40.19 (O7)
- net ADDR_EN: now also U36.1 (OE), U41.1 (OE)
- no-connect marks 17 -> 15
Changed lines of the file:
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@@
   (no_connect (at 275.59 31.115))
   (no_connect (at 223.52 31.115))
-  (no_connect (at 275.59 46.355))
   (no_connect (at 275.59 28.575))
   (no_connect (at 223.52 28.575))
@@
   (no_connect (at 146.685 187.325))
   (no_connect (at 250.19 31.115))
-  (no_connect (at 250.19 46.355))
   (no_connect (at 198.12 31.115))
   (no_connect (at 198.12 28.575))
@@
     (effects (font (size 1.27 1.27)) (justify right bottom))
   )
-  (label "D3" (at 180.34 40.64 0)
+  (label "D3" (at 180.34 101.6 0)
     (effects (font (size 1.27 1.27)) (justify left bottom))
   )
@@
     (effects (font (size 1.27 1.27)) (justify left bottom))
   )
-  (label "A3" (at 180.34 43.18 0)
+  (label "A3" (at 180.34 38.1 0)
     (effects (font (size 1.27 1.27)) (justify left bottom))
   )
@@
     (effects (font (size 1.27 1.27)) (justify left bottom))
   )
-  (label "D7" (at 180.34 38.1 0)
+  (label "D7" (at 180.34 91.44 0)
     (effects (font (size 1.27 1.27)) (justify left bottom))
   )
@@
     (effects (font (size 1.27 1.27)) (justify left bottom))
   )
+  (label "ADDR_EN" (at 275.59 46.355 0)
+    (effects (font (size 1.27 1.27)) (justify left bottom))
+  )
   (label "D7" (at 44.45 59.69 180)
     (effects (font (size 1.27 1.27)) (justify right bottom))
@@
     (effects (font (size 1.27 1.27)) (justify left bottom))
   )
-  (label "A6" (at 180.34 91.44 0)
-    (effects (font (size 1.27 1.27)) (justify left bottom))
-  )
-  (label "D0" (at 180.34 27.94 0)
+  (label "A6" (at 180.34 40.64 0)
+    (effects (font (size 1.27 1.27)) (justify left bottom))
+  )
+  (label "D0" (at 180.34 86.36 0)
     (effects (font (size 1.27 1.27)) (justify left bottom))
   )
@@
     (effects (font (size 1.27 1.27)) (justify right bottom))
   )
+  (label "ADDR_EN" (at 250.19 109.22 180)
+    (effects (font (size 1.27 1.27)) (justify right bottom))
+  )
+  (label "ADDR_EN" (at 154.94 53.34 180)
+    (effects (font (size 1.27 1.27)) (justify right bottom))
+  )
   (label "RESET_P_DRIVE" (at 34.925 160.655 180)
     (effects (font (size 1.27 1.27)) (justify right bottom))
@@
     (effects (font (size 1.27 1.27)) (justify left bottom))
   )
-  (label "A2" (at 180.34 86.36 0)
+  (label "A2" (at 180.34 27.94 0)
     (effects (font (size 1.27 1.27)) (justify left bottom))
   )
@@
     (effects (font (size 1.27 1.27)) (justify right bottom))
   )
+  (label "R_W" (at 154.94 109.22 180)
+    (effects (font (size 1.27 1.27)) (justify right bottom))
+  )
   (label "A5" (at 180.34 33.02 0)
     (effects (font (size 1.27 1.27)) (justify left bottom))
@@
     (effects (font (size 1.27 1.27)) (justify left bottom))
   )
-  (label "A0" (at 180.34 101.6 0)
+  (label "A0" (at 180.34 43.18 0)
     (effects (font (size 1.27 1.27)) (justify left bottom))
   )
@@
     (effects (font (size 1.27 1.27)) (justify right))
     (property "Intersheet References" "${INTERSHEET_REFS}" (id 0) (at 142.4879 147.2406 0)
+      (effects (font (size 1.27 1.27)) (justify right) hide)
+    )
+  )
+  (global_label "MUX_DO7" (shape input) (at 250.19 45.72 180) (fields_autoplaced)
+    (effects (font (size 1.27 1.27)) (justify right))
+    (property "Intersheet References" "${INTERSHEET_REFS}" (id 0) (at 239.0079 45.6406 0)
       (effects (font (size 1.27 1.27)) (justify right) hide)
     )
@@
     )
     (pin "1")
-  )
-  (symbol (lib_id "Device:R_Network08") (at 35.56 67.31 90) (unit 1)
-    (in_bom yes) (on_board yes)
-    (property "Reference" "RN3" (id 0) (at 29.21 60.96 90))
-    (property "Value" "3.3K x 8" (id 1) (at 30.48 67.31 0))
-    (property "Footprint" "Resistor_THT:R_Array_SIP9" (id 2) (at 35.56 55.245 90)
-      (effects (font (size 1.27 1.27)) hide)
-    )
-    (property "Datasheet" "http://www.vishay.com/docs/31509/csc.pdf" (id 3) (at 35.56 67.31 0)
-      (effects (font (size 1.27 1.27)) hide)
-    )
-    (pin "1")
-    (pin "2")
-    (pin "3")
-    (pin "4")
-    (pin "5")
-    (pin "6")
-    (pin "7")
-    (pin "8")
-    (pin "9")
-  )
-  (symbol (lib_id "Device:R_Network08") (at 66.04 67.31 270) (mirror x) (unit 1)
-    (in_bom yes) (on_board yes)
-    (property "Reference" "RN6" (id 0) (at 72.39 60.96 90))
-    (property "Value" "3.3K x 8" (id 1) (at 71.12 68.58 0))
-    (property "Footprint" "Resistor_THT:R_Array_SIP9" (id 2) (at 66.04 55.245 90)
-      (effects (font (size 1.27 1.27)) hide)
-    )
-    (property "Datasheet" "http://www.vishay.com/docs/31509/csc.pdf" (id 3) (at 66.04 67.31 0)
-      (effects (font (size 1.27 1.27)) hide)
-    )
-    (pin "1")
-    (pin "2")
-    (pin "3")
-    (pin "4")
-    (pin "5")
-    (pin "6")
-    (pin "7")
-    (pin "8")
-    (pin "9")
   )
   (symbol (lib_id "power:+3.3V") (at 116.205 76.2 0) (unit 1)
@@
     )
     (property "Datasheet" "" (id 3) (at 167.64 116.84 0)
-      (effects (font (size 1.27 1.27)) hide)
-    )
-    (pin "1")
-  )
-  (symbol (lib_id "power:GND") (at 154.94 53.34 0) (unit 1)
-    (in_bom yes) (on_board yes) (fields_autoplaced)
-    (property "Reference" "#PWR0261" (id 0) (at 154.94 59.69 0)
-      (effects (font (size 1.27 1.27)) hide)
-    )
-    (property "Value" "GND" (id 1) (at 154.94 58.42 0))
-    (property "Footprint" "" (id 2) (at 154.94 53.34 0)
-      (effects (font (size 1.27 1.27)) hide)
-    )
-    (property "Datasheet" "" (id 3) (at 154.94 53.34 0)
       (effects (font (size 1.27 1.27)) hide)
     )
@@
     (pin "Z")
   )
-  (symbol (lib_id "Device:R_Network08") (at 66.04 46.99 270) (mirror x) (unit 1)
-    (in_bom yes) (on_board yes)
-    (property "Reference" "RN5" (id 0) (at 72.39 54.61 90))
-    (property "Value" "3.3K x 8" (id 1) (at 71.12 46.99 0))
-    (property "Footprint" "Resistor_THT:R_Array_SIP9" (id 2) (at 66.04 34.925 90)
-      (effects (font (size 1.27 1.27)) hide)
-    )
-    (property "Datasheet" "http://www.vishay.com/docs/31509/csc.pdf" (id 3) (at 66.04 46.99 0)
-      (effects (font (size 1.27 1.27)) hide)
-    )
-    (pin "1")
-    (pin "2")
-    (pin "3")
-    (pin "4")
-    (pin "5")
-    (pin "6")
-    (pin "7")
-    (pin "8")
-    (pin "9")
-  )
   (symbol (lib_id "power:GND") (at 210.82 61.595 0) (unit 1)
     (in_bom yes) (on_board yes) (fields_autoplaced)
@@
     )
     (property "Datasheet" "" (id 3) (at 116.205 61.595 0)
-      (effects (font (size 1.27 1.27)) hide)
-    )
-    (pin "1")
-  )
-  (symbol (lib_id "power:+5V") (at 71.12 77.47 0) (unit 1)
-    (in_bom yes) (on_board yes) (fields_autoplaced)
-    (property "Reference" "#PWR0238" (id 0) (at 71.12 81.28 0)
-      (effects (font (size 1.27 1.27)) hide)
-    )
-    (property "Value" "+5V" (id 1) (at 71.12 72.39 0))
-    (property "Footprint" "" (id 2) (at 71.12 77.47 0)
-      (effects (font (size 1.27 1.27)) hide)
-    )
-    (property "Datasheet" "" (id 3) (at 71.12 77.47 0)
       (effects (font (size 1.27 1.27)) hide)
     )
@@
     (pin "9")
   )
-  (symbol (lib_id "power:+5V") (at 30.48 77.47 0) (unit 1)
-    (in_bom yes) (on_board yes) (fields_autoplaced)
-    (property "Reference" "#PWR0241" (id 0) (at 30.48 81.28 0)
-      (effects (font (size 1.27 1.27)) hide)
-    )
-    (property "Value" "+5V" (id 1) (at 30.48 72.39 0))
-    (property "Footprint" "" (id 2) (at 30.48 77.47 0)
-      (effects (font (size 1.27 1.27)) hide)
-    )
-    (property "Datasheet" "" (id 3) (at 30.48 77.47 0)
-      (effects (font (size 1.27 1.27)) hide)
-    )
-    (pin "1")
-  )
-  (symbol (lib_id "power:+5V") (at 71.12 57.15 0) (unit 1)
-    (in_bom yes) (on_board yes) (fields_autoplaced)
-    (property "Reference" "#PWR0248" (id 0) (at 71.12 60.96 0)
-      (effects (font (size 1.27 1.27)) hide)
-    )
-    (property "Value" "+5V" (id 1) (at 71.12 52.07 0))
-    (property "Footprint" "" (id 2) (at 71.12 57.15 0)
-      (effects (font (size 1.27 1.27)) hide)
-    )
-    (property "Datasheet" "" (id 3) (at 71.12 57.15 0)
-      (effects (font (size 1.27 1.27)) hide)
-    )
-    (pin "1")
-  )
   (symbol (lib_id "power:+5V") (at 22.86 52.07 0) (unit 1)
     (in_bom yes) (on_board yes) (fields_autoplaced)
@@
     (pin "11")
   )
-  (symbol (lib_id "power:GND") (at 154.94 109.22 0) (unit 1)
-    (in_bom yes) (on_board yes) (fields_autoplaced)
-    (property "Reference" "#PWR0263" (id 0) (at 154.94 115.57 0)
-      (effects (font (size 1.27 1.27)) hide)
-    )
-    (property "Value" "GND" (id 1) (at 154.94 114.3 0))
-    (property "Footprint" "" (id 2) (at 154.94 109.22 0)
-      (effects (font (size 1.27 1.27)) hide)
-    )
-    (property "Datasheet" "" (id 3) (at 154.94 109.22 0)
-      (effects (font (size 1.27 1.27)) hide)
-    )
-    (pin "1")
-  )
   (symbol (lib_id "74xx:74LS374") (at 262.89 41.275 0) (unit 1)
     (in_bom yes) (on_board yes) (fields_autoplaced)
@@
     (pin "9")
   )
-  (symbol (lib_id "power:GND") (at 250.19 109.22 0) (unit 1)
-    (in_bom yes) (on_board yes) (fields_autoplaced)
-    (property "Reference" "#PWR0279" (id 0) (at 250.19 115.57 0)
-      (effects (font (size 1.27 1.27)) hide)
-    )
-    (property "Value" "GND" (id 1) (at 250.19 114.3 0))
-    (property "Footprint" "" (id 2) (at 250.19 109.22 0)
-      (effects (font (size 1.27 1.27)) hide)
-    )
-    (property "Datasheet" "" (id 3) (at 250.19 109.22 0)
-      (effects (font (size 1.27 1.27)) hide)
-    )
-    (pin "1")
-  )
   (symbol (lib_id "Device:R_Network08") (at 27.94 41.91 90) (unit 1)
